File: Hardware/SparkFun_HSTX_to_DVI_Breakout.kicad_sch (KiCad schematic)
At the start: 22 parts, among them J1 Conn_01x22_FPC_0.5mm_RA, J2 HDMI, Q1 BSS138, U1 AP3602

Commit message: Add dates
Parts:
- J2: PROD_ID (none) -> CONN-25635
Changed lines of the file:
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@@
 	(title_block
 		(title "SparkFun HSTX to DVI Breakout")
+		(date "2025-03-03")
 		(rev "v10")
 		(company "SparkFun Electronics")
@@
 			(effects
 				(font
+					(size 1.27 1.27)
+				)
+				(hide yes)
+			)
+		)
+		(property "PROD_ID" "CONN-25635"
+			(at 254.254 130.556 0)
+			(effects
+				(font

Commit message: Update prod_id
Parts:
- Q1: PROD_ID TRANS-25647 -> TRANS-25637
Changed lines of the file:
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@@
 			)
 		)
-		(property "PROD_ID" "TRANS-25647"
+		(property "PROD_ID" "TRANS-25637"
 			(at 35.56 181.61 0)
 			(effects
@@
 	)
 	(symbol
-		(lib_name "Q_NMOS_0.2A_50V_DUAL_1")
 		(lib_id "SparkFun-DiscreteSemi:Q_NMOS_0.2A_50V_DUAL")
 		(at 50.8 156.21 270)
@@
 			)
 		)
-		(property "PROD_ID" "TRANS-25647"
+		(property "PROD_ID" "TRANS-25637"
 			(at 35.56 156.21 0)
 			(effects
